Commit message: chore: attach marker holder link to elfin robot definition

File: elfin10_l/elfin10_l_ros2_gazebo/urdf/elfin10_l.urdf.xacro (robot description, xacro)
@@ -439,13 +439,31 @@
       xyz="0 0 0" />
   </joint>
- <link name="elfin_dummy_gripper"/>
-  <joint name="elfin_dummy_joint" type="fixed">
-    <origin
-      xyz="0 0.109 0"
-      rpy="-1.5708 -1.5708 0" />
-    <parent
-      link="elfin_link6" />
-    <child
-      link="elfin_dummy_gripper" />
+  <link name="marker_holder_link">
+    <visual>
+      <origin xyz="0 0 0" rpy="0 0 0"/>
+      <geometry>
+        <mesh filename="file://$(find surface_tracking_visualization)/meshes/marker_holder.stl" scale="0.001 0.001 0.001"/>
+      </geometry>
+      <material name="white">
+        <color rgba="1 1 1 1" />
+      </material>
+    </visual>
+    <collision>
+      <origin xyz="0 0 0" rpy="0 0 0"/>
+      <geometry>
+        <mesh filename="file://$(find surface_tracking_visualization)/meshes/marker_holder.stl" scale="0.001 0.001 0.001"/>
+      </geometry>
+    </collision>
+  </link>
+  <joint name="flange_to_holder_joint" type="fixed">
+    <parent link="elfin_end_link" />
+    <child link="marker_holder_link" />
+    <origin xyz="0 0 0" rpy="0 0 -1.16937" />
+  </joint>
+  <link name="pen_tip_link"/>
+  <joint name="holder_to_pen_tip_joint" type="fixed">
+    <parent link="marker_holder_link" />
+    <child link="pen_tip_link" />
+    <origin xyz="0 0 0.15" rpy="0 0 0" />
   </joint>
 </robot>

File: elfin_description/urdf/elfin10_l.urdf.xacro (robot description, xacro)
@@ -426,13 +426,31 @@
       xyz="0 0 0" />
   </joint>
-  <link name="elfin_dummy_gripper"/>
-  <joint name="elfin_dummy_joint" type="fixed">
-    <origin
-      xyz="0 0.109 0"
-      rpy="-1.5708 -1.5708 0" />
-    <parent
-      link="elfin_link6" />
-    <child
-      link="elfin_dummy_gripper" />
+  <link name="marker_holder_link">
+    <visual>
+      <origin xyz="0 0 0" rpy="0 0 0"/>
+      <geometry>
+        <mesh filename="file://$(find surface_tracking_visualization)/meshes/marker_holder.stl" scale="0.001 0.001 0.001"/>
+      </geometry>
+      <material name="white">
+        <color rgba="1 1 1 1" />
+      </material>
+    </visual>
+    <collision>
+      <origin xyz="0 0 0" rpy="0 0 0"/>
+      <geometry>
+        <mesh filename="file://$(find surface_tracking_visualization)/meshes/marker_holder.stl" scale="0.001 0.001 0.001"/>
+      </geometry>
+    </collision>
+  </link>
+  <joint name="flange_to_holder_joint" type="fixed">
+    <parent link="elfin_end_link" />
+    <child link="marker_holder_link" />
+    <origin xyz="0 0 0" rpy="0 0 -1.16937" />
+  </joint>
+  <link name="pen_tip_link"/>
+  <joint name="holder_to_pen_tip_joint" type="fixed">
+    <parent link="marker_holder_link" />
+    <child link="pen_tip_link" />
+    <origin xyz="0 0 0.15" rpy="0 0 0" />
   </joint>
 </robot>

Commit message: chore: attach tip link, change marker holder link to the new compliance end effector

File: elfin10_l/elfin10_l_ros2_gazebo/urdf/elfin10_l.urdf.xacro (robot description, xacro)
@@ -443,5 +443,5 @@
       <origin xyz="0 0 0" rpy="0 0 0"/>
       <geometry>
-        <mesh filename="file://$(find surface_tracking_visualization)/meshes/marker_holder.stl" scale="0.001 0.001 0.001"/>
+        <mesh filename="file://$(find surface_tracking_visualization)/meshes/marker_holder_comply.stl" scale="0.001 0.001 0.001"/>
       </geometry>
       <material name="white">
@@ -452,5 +452,5 @@
       <origin xyz="0 0 0" rpy="0 0 0"/>
       <geometry>
-        <mesh filename="file://$(find surface_tracking_visualization)/meshes/marker_holder.stl" scale="0.001 0.001 0.001"/>
+        <mesh filename="file://$(find surface_tracking_visualization)/meshes/marker_holder_comply.stl" scale="0.001 0.001 0.001"/>
       </geometry>
     </collision>
@@ -459,11 +459,27 @@
     <parent link="elfin_end_link" />
     <child link="marker_holder_link" />
-    <origin xyz="0 0 0" rpy="0 0 -1.16937" />
-  </joint>
-  <link name="pen_tip_link"/>
+    <origin xyz="0 0 0" rpy="0 0 1.972222654" />
+  </joint>
+  <link name="pen_tip_link">
+    <visual>
+      <origin xyz="0 0 0.07" rpy="0 0 0"/>
+      <geometry>
+        <cylinder radius="0.0075" length="0.14"/>
+      </geometry>
+      <material name="white">
+        <color rgba="1 1 1 1" />
+      </material>
+    </visual>
+    <collision>
+      <origin xyz="0 0 0.07" rpy="0 0 0"/>
+      <geometry>
+        <cylinder radius="0.0075" length="0.14"/>
+      </geometry>
+    </collision>
+  </link>
   <joint name="holder_to_pen_tip_joint" type="fixed">
     <parent link="marker_holder_link" />
     <child link="pen_tip_link" />
-    <origin xyz="0 0 0.15" rpy="0 0 0" />
+    <origin xyz="0 -0.113 0.0695" rpy="-1.57 3.14 0" />
   </joint>
 </robot>

File: elfin_description/urdf/elfin10_l.urdf.xacro (robot description, xacro)
@@ -430,5 +430,5 @@
       <origin xyz="0 0 0" rpy="0 0 0"/>
       <geometry>
-        <mesh filename="file://$(find surface_tracking_visualization)/meshes/marker_holder.stl" scale="0.001 0.001 0.001"/>
+        <mesh filename="file://$(find surface_tracking_visualization)/meshes/marker_holder_comply.stl" scale="0.001 0.001 0.001"/>
       </geometry>
       <material name="white">
@@ -439,5 +439,5 @@
       <origin xyz="0 0 0" rpy="0 0 0"/>
       <geometry>
-        <mesh filename="file://$(find surface_tracking_visualization)/meshes/marker_holder.stl" scale="0.001 0.001 0.001"/>
+        <mesh filename="file://$(find surface_tracking_visualization)/meshes/marker_holder_comply.stl" scale="0.001 0.001 0.001"/>
       </geometry>
     </collision>
@@ -446,11 +446,27 @@
     <parent link="elfin_end_link" />
     <child link="marker_holder_link" />
-    <origin xyz="0 0 0" rpy="0 0 -1.16937" />
-  </joint>
-  <link name="pen_tip_link"/>
+    <origin xyz="0 0 0" rpy="0 0 1.972222654" />
+  </joint>
+  <link name="pen_tip_link">
+    <visual>
+      <origin xyz="0 0 0.07" rpy="0 0 0"/>
+      <geometry>
+        <cylinder radius="0.0075" length="0.14"/>
+      </geometry>
+      <material name="white">
+        <color rgba="1 1 1 1" />
+      </material>
+    </visual>
+    <collision>
+      <origin xyz="0 0 0.07" rpy="0 0 0"/>
+      <geometry>
+        <cylinder radius="0.0075" length="0.14"/>
+      </geometry>
+    </collision>
+  </link>
   <joint name="holder_to_pen_tip_joint" type="fixed">
     <parent link="marker_holder_link" />
     <child link="pen_tip_link" />
-    <origin xyz="0 0 0.15" rpy="0 0 0" />
+    <origin xyz="0 -0.113 0.0695" rpy="-1.57 3.14 0" />
   </joint>
 </robot>
